Commit message: fix(sim): level chassis and raise lidar for a clean horizontal scan
- Lower head tube 0.098 m so the front wheel reaches the ground like the rear;
  robot was resting ~4.2 deg nose-down, tilting the lidar into the floor and
  producing a phantom obstacle in the front cone.
- Raise lidar 0.10 m above the control-panel/front-camera assembly, which was
  clipping the scan plane at ~0.83 m.
Result: /etrike/scan is now horizontal and unobstructed.

File: bglx_ws/src/etrike_description/urdf/components/frame.xacro (robot description, xacro)
@@ -226,5 +226,5 @@
       <child link="frame_head_tube"/>
       <!-- Raised up so fork+wheel reaches ground -->
-      <origin xyz="1.0 0 0.20" rpy="0 0 0"/>
+      <origin xyz="1.0 0 0.102" rpy="0 0 0"/>
     </joint>
     <!-- ============================================================== -->

File: bglx_ws/src/etrike_description/urdf/components/sensors.xacro (robot description, xacro)
@@ -32,5 +32,5 @@
       <parent link="sensor_mount_plate"/>
       <child link="lidar_base"/>
-      <origin xyz="0 0 0.02" rpy="0 0 0"/>
+      <origin xyz="0 0 0.12" rpy="0 0 0"/>
     </joint>
     <link name="lidar_sensor">
