Commit message: perf(sim): remove unused side cameras to free CPU
Nav2's control loop was missing its 20 Hz rate and stalling on turns because
four RGB cameras rendered every frame. The side cameras aren't used by
navigation, so remove their links, joints, and Gazebo sensors. Front, ground,
depth, and lidar remain.

File: bglx_ws/src/etrike_description/urdf/components/sensors.xacro (robot description, xacro)
@@ -149,60 +149,8 @@
     <!-- SIDE LEFT CAMERA - 90° for lane monitoring                     -->
     <!-- ============================================================== -->
-    <link name="camera_side_left">
-      <inertial>
-        <mass value="0.08"/>
-        <origin xyz="0 0 0" rpy="0 0 0"/>
-        <xacro:box_inertia m="0.08" x="0.025" y="0.025" z="0.025"/>
-      </inertial>
-      <visual>
-        <origin xyz="0 0 0" rpy="0 0 0"/>
-        <geometry>
-          <box size="0.025 0.025 0.025"/>
-        </geometry>
-        <material name="carbon_fiber"/>
-      </visual>
-      <collision>
-        <origin xyz="0 0 0" rpy="0 0 0"/>
-        <geometry>
-          <box size="0.025 0.025 0.025"/>
-        </geometry>
-      </collision>
-    </link>
-    <joint name="camera_side_left_joint" type="fixed">
-      <parent link="cargo_box"/>
-      <child link="camera_side_left"/>
-      <!-- Left side center, pointing 90° left -->
-      <origin xyz="0 0.24 0.10" rpy="0 0 1.5708"/>
-    </joint>
-    <!-- ============================================================== -->
+<!-- ============================================================== -->
     <!-- SIDE RIGHT CAMERA - 90° for lane monitoring                    -->
     <!-- ============================================================== -->
-    <link name="camera_side_right">
-      <inertial>
-        <mass value="0.08"/>
-        <origin xyz="0 0 0" rpy="0 0 0"/>
-        <xacro:box_inertia m="0.08" x="0.025" y="0.025" z="0.025"/>
-      </inertial>
-      <visual>
-        <origin xyz="0 0 0" rpy="0 0 0"/>
-        <geometry>
-          <box size="0.025 0.025 0.025"/>
-        </geometry>
-        <material name="carbon_fiber"/>
-      </visual>
-      <collision>
-        <origin xyz="0 0 0" rpy="0 0 0"/>
-        <geometry>
-          <box size="0.025 0.025 0.025"/>
-        </geometry>
-      </collision>
-    </link>
-    <joint name="camera_side_right_joint" type="fixed">
-      <parent link="cargo_box"/>
-      <child link="camera_side_right"/>
-      <!-- Right side center, pointing 90° right -->
-      <origin xyz="0 -0.24 0.10" rpy="0 0 -1.5708"/>
-    </joint>
-    <!-- ============================================================== -->
+<!-- ============================================================== -->
     <!-- REAR LEFT CAMERA - 135° for blind spot coverage                -->
     <!-- ============================================================== -->

File: bglx_ws/src/etrike_description/urdf/gazebo/gazebo_config.xacro (robot description, xacro)
@@ -26,7 +26,5 @@
   <gazebo reference="camera_front_left"><material>Gazebo/Black</material></gazebo>
   <gazebo reference="camera_front_right"><material>Gazebo/Black</material></gazebo>
-  <gazebo reference="camera_side_left"><material>Gazebo/Black</material></gazebo>
-  <gazebo reference="camera_side_right"><material>Gazebo/Black</material></gazebo>
-  <gazebo reference="camera_rear_left"><material>Gazebo/Black</material></gazebo>
+<gazebo reference="camera_rear_left"><material>Gazebo/Black</material></gazebo>
   <gazebo reference="camera_rear_right"><material>Gazebo/Black</material></gazebo>
   <gazebo reference="camera_rear_main"><material>Gazebo/Black</material></gazebo>
@@ -178,64 +176,8 @@
   <!-- LEFT CAMERA - Side view for turning                            -->
   <!-- ============================================================== -->
-  <gazebo reference="camera_side_left">
-    <sensor name="camera_left" type="camera">
-      <always_on>true</always_on>
-      <visualize>true</visualize>
-      <update_rate>20</update_rate>
-      <camera name="left">
-        <horizontal_fov>1.5708</horizontal_fov>
-        <image>
-          <width>640</width>
-          <height>480</height>
-          <format>R8G8B8</format>
-        </image>
-        <clip>
-          <near>0.1</near>
-          <far>50</far>
-        </clip>
-      </camera>
-      <plugin name="camera_left_controller" filename="libgazebo_ros_camera.so">
-        <ros>
-          <namespace>/etrike</namespace>
-          <remapping>image_raw:=camera/left/image_raw</remapping>
-          <remapping>camera_info:=camera/left/camera_info</remapping>
-        </ros>
-        <camera_name>left</camera_name>
-        <frame_name>camera_side_left</frame_name>
-      </plugin>
-    </sensor>
-  </gazebo>
-  <!-- ============================================================== -->
+<!-- ============================================================== -->
   <!-- RIGHT CAMERA - Side view for turning                           -->
   <!-- ============================================================== -->
-  <gazebo reference="camera_side_right">
-    <sensor name="camera_right" type="camera">
-      <always_on>true</always_on>
-      <visualize>true</visualize>
-      <update_rate>20</update_rate>
-      <camera name="right">
-        <horizontal_fov>1.5708</horizontal_fov>
-        <image>
-          <width>640</width>
-          <height>480</height>
-          <format>R8G8B8</format>
-        </image>
-        <clip>
-          <near>0.1</near>
-          <far>50</far>
-        </clip>
-      </camera>
-      <plugin name="camera_right_controller" filename="libgazebo_ros_camera.so">
-        <ros>
-          <namespace>/etrike</namespace>
-          <remapping>image_raw:=camera/right/image_raw</remapping>
-          <remapping>camera_info:=camera/right/camera_info</remapping>
-        </ros>
-        <camera_name>right</camera_name>
-        <frame_name>camera_side_right</frame_name>
-      </plugin>
-    </sensor>
-  </gazebo>
-  <!-- ============================================================== -->
+<!-- ============================================================== -->
   <!-- GROUND CAMERA - Close obstacle detection                       -->
   <!-- ============================================================== -->
