Commit message: style(sim): wheels with rims/hubs, BGLX accent stripes, clean fork
Visual-only (no joints/collisions/mounts changed, TF tree intact):
- rear + front wheels get spinning rim + hubcap sub-links
- cargo box gets BGLX-green accent stripes (sides + front)
- steering_link rebuilt as a clean telescoping fork (steerer, legs, axle)

File: bglx_ws/src/etrike_description/urdf/components/cargo_box.xacro (robot description, xacro)
@@ -124,4 +124,41 @@
       <origin xyz="0 0 0.02" rpy="0 0 0"/>
     </joint>
+    <!-- ==== BGLX accent stripes (visual only) ==== -->
+    <link name="accent_left">
+      <inertial><mass value="0.01"/><origin xyz="0 0 0" rpy="0 0 0"/>
+        <inertia ixx="1e-6" ixy="0" ixz="0" iyy="1e-6" iyz="0" izz="1e-6"/></inertial>
+      <visual><origin xyz="0 0 0" rpy="0 0 0"/>
+        <geometry><box size="0.50 0.014 0.05"/></geometry>
+        <material name="bglx_green"/></visual>
+    </link>
+    <joint name="accent_left_joint" type="fixed">
+      <parent link="cargo_box"/><child link="accent_left"/>
+      <origin xyz="0 0.229 -0.10" rpy="0 0 0"/>
+    </joint>
+    <gazebo reference="accent_left"><material>Gazebo/Green</material></gazebo>
+    <link name="accent_right">
+      <inertial><mass value="0.01"/><origin xyz="0 0 0" rpy="0 0 0"/>
+        <inertia ixx="1e-6" ixy="0" ixz="0" iyy="1e-6" iyz="0" izz="1e-6"/></inertial>
+      <visual><origin xyz="0 0 0" rpy="0 0 0"/>
+        <geometry><box size="0.50 0.014 0.05"/></geometry>
+        <material name="bglx_green"/></visual>
+    </link>
+    <joint name="accent_right_joint" type="fixed">
+      <parent link="cargo_box"/><child link="accent_right"/>
+      <origin xyz="0 -0.229 -0.10" rpy="0 0 0"/>
+    </joint>
+    <gazebo reference="accent_right"><material>Gazebo/Green</material></gazebo>
+    <link name="accent_front">
+      <inertial><mass value="0.01"/><origin xyz="0 0 0" rpy="0 0 0"/>
+        <inertia ixx="1e-6" ixy="0" ixz="0" iyy="1e-6" iyz="0" izz="1e-6"/></inertial>
+      <visual><origin xyz="0 0 0" rpy="0 0 0"/>
+        <geometry><box size="0.014 0.40 0.05"/></geometry>
+        <material name="bglx_green"/></visual>
+    </link>
+    <joint name="accent_front_joint" type="fixed">
+      <parent link="cargo_box"/><child link="accent_front"/>
+      <origin xyz="0.281 0 -0.10" rpy="0 0 0"/>
+    </joint>
+    <gazebo reference="accent_front"><material>Gazebo/Green</material></gazebo>
   </xacro:macro>
 </robot>

File: bglx_ws/src/etrike_description/urdf/components/front_fork.xacro (robot description, xacro)
@@ -48,59 +48,32 @@
         <xacro:box_inertia m="1.0" x="0.04" y="0.10" z="0.25"/>
       </inertial>
-      <!-- Fork stem -->
       <visual>
-        <origin xyz="0.02 0 -0.05" rpy="0 0.2 0"/>
-        <geometry>
-          <cylinder radius="0.015" length="0.12"/>
-        </geometry>
+        <origin xyz="0.02 0 -0.04" rpy="0 0 0"/>
+        <geometry><cylinder radius="0.022" length="0.12"/></geometry>
+        <material name="fork"/>
+      </visual>
+      <visual>
+        <origin xyz="0.035 0 -0.05" rpy="0 0 0"/>
+        <geometry><box size="0.05 0.13 0.04"/></geometry>
+        <material name="fork"/>
+      </visual>
+      <visual>
+        <origin xyz="0.04 0.055 -0.17" rpy="0 0 0"/>
+        <geometry><cylinder radius="0.016" length="0.26"/></geometry>
+        <material name="fork"/>
+      </visual>
+      <visual>
+        <origin xyz="0.04 -0.055 -0.17" rpy="0 0 0"/>
+        <geometry><cylinder radius="0.016" length="0.26"/></geometry>
+        <material name="fork"/>
+      </visual>
+      <visual>
+        <origin xyz="0.04 0 -0.28" rpy="1.5708 0 0"/>
+        <geometry><cylinder radius="0.014" length="0.14"/></geometry>
         <material name="fork"/>
       </visual>
       <collision>
-        <origin xyz="0.02 0 -0.05" rpy="0 0.2 0"/>
-        <geometry>
-          <cylinder radius="0.015" length="0.12"/>
-        </geometry>
-      </collision>
-      <!-- Left fork tube -->
-      <visual>
-        <origin xyz="0.04 0.04 -0.18" rpy="0 0 0"/>
-        <geometry>
-          <cylinder radius="0.015" length="0.20"/>
-        </geometry>
-        <material name="fork"/>
-      </visual>
-      <collision>
-        <origin xyz="0.04 0.04 -0.18" rpy="0 0 0"/>
-        <geometry>
-          <cylinder radius="0.015" length="0.20"/>
-        </geometry>
-      </collision>
-      <!-- Right fork tube -->
-      <visual>
-        <origin xyz="0.04 -0.04 -0.18" rpy="0 0 0"/>
-        <geometry>
-          <cylinder radius="0.015" length="0.20"/>
-        </geometry>
-        <material name="fork"/>
-      </visual>
-      <collision>
-        <origin xyz="0.04 -0.04 -0.18" rpy="0 0 0"/>
-        <geometry>
-          <cylinder radius="0.015" length="0.20"/>
-        </geometry>
-      </collision>
-      <!-- Axle bridge -->
-      <visual>
-        <origin xyz="0.04 0 -0.28" rpy="${pi/2} 0 0"/>
-        <geometry>
-          <cylinder radius="0.012" length="0.08"/>
-        </geometry>
-        <material name="fork"/>
-      </visual>
-      <collision>
-        <origin xyz="0.04 0 -0.28" rpy="${pi/2} 0 0"/>
-        <geometry>
-          <cylinder radius="0.012" length="0.08"/>
-        </geometry>
+        <origin xyz="0.035 0 -0.14" rpy="0 0 0"/>
+        <geometry><box size="0.05 0.14 0.26"/></geometry>
       </collision>
     </link>
@@ -142,4 +115,28 @@
       <dynamics damping="0.001" friction="0.001"/>
     </joint>
+    <link name="front_rim">
+      <inertial><mass value="0.2"/><origin xyz="0 0 0" rpy="0 0 0"/>
+        <inertia ixx="1e-4" ixy="0" ixz="0" iyy="1e-4" iyz="0" izz="1e-4"/></inertial>
+      <visual><origin xyz="0 0 0" rpy="${pi/2} 0 0"/>
+        <geometry><cylinder radius="0.11" length="0.052"/></geometry>
+        <material name="aluminum"/></visual>
+    </link>
+    <joint name="front_rim_joint" type="fixed">
+      <parent link="front_wheel"/><child link="front_rim"/>
+      <origin xyz="0 0 0" rpy="0 0 0"/>
+    </joint>
+    <gazebo reference="front_rim"><material>Gazebo/Grey</material></gazebo>
+    <link name="front_hubcap">
+      <inertial><mass value="0.05"/><origin xyz="0 0 0" rpy="0 0 0"/>
+        <inertia ixx="1e-5" ixy="0" ixz="0" iyy="1e-5" iyz="0" izz="1e-5"/></inertial>
+      <visual><origin xyz="0 0 0" rpy="${pi/2} 0 0"/>
+        <geometry><cylinder radius="0.045" length="0.062"/></geometry>
+        <material name="hub_motor"/></visual>
+    </link>
+    <joint name="front_hubcap_joint" type="fixed">
+      <parent link="front_wheel"/><child link="front_hubcap"/>
+      <origin xyz="0 0 0" rpy="0 0 0"/>
+    </joint>
+    <gazebo reference="front_hubcap"><material>Gazebo/DarkGrey</material></gazebo>
   </xacro:macro>
 </robot>

File: bglx_ws/src/etrike_description/urdf/components/rear_drive.xacro (robot description, xacro)
@@ -127,4 +127,28 @@
       <dynamics damping="0.1" friction="0.05"/>
     </joint>
+    <link name="${prefix}_rim">
+      <inertial><mass value="0.2"/><origin xyz="0 0 0" rpy="0 0 0"/>
+        <inertia ixx="1e-4" ixy="0" ixz="0" iyy="1e-4" iyz="0" izz="1e-4"/></inertial>
+      <visual><origin xyz="0 0 0" rpy="${pi/2} 0 0"/>
+        <geometry><cylinder radius="0.11" length="0.062"/></geometry>
+        <material name="aluminum"/></visual>
+    </link>
+    <joint name="${prefix}_rim_joint" type="fixed">
+      <parent link="${prefix}_wheel"/><child link="${prefix}_rim"/>
+      <origin xyz="0 0 0" rpy="0 0 0"/>
+    </joint>
+    <gazebo reference="${prefix}_rim"><material>Gazebo/Grey</material></gazebo>
+    <link name="${prefix}_hubcap">
+      <inertial><mass value="0.05"/><origin xyz="0 0 0" rpy="0 0 0"/>
+        <inertia ixx="1e-5" ixy="0" ixz="0" iyy="1e-5" iyz="0" izz="1e-5"/></inertial>
+      <visual><origin xyz="0 0 0" rpy="${pi/2} 0 0"/>
+        <geometry><cylinder radius="0.045" length="0.072"/></geometry>
+        <material name="hub_motor"/></visual>
+    </link>
+    <joint name="${prefix}_hubcap_joint" type="fixed">
+      <parent link="${prefix}_wheel"/><child link="${prefix}_hubcap"/>
+      <origin xyz="0 0 0" rpy="0 0 0"/>
+    </joint>
+    <gazebo reference="${prefix}_hubcap"><material>Gazebo/DarkGrey</material></gazebo>
   </xacro:macro>
   <!-- Main macro that creates both rear wheels -->
