Commit message: feat(sim): ros2_control tricycle_steering_controller for the trike

File: bglx_ws/src/etrike_description/urdf/components/front_fork.xacro (robot description, xacro)
@@ -2,13 +2,23 @@
 <robot xmlns:xacro="http://www.ros.org/wiki/xacro">
   <!-- ================================================================== -->
-  <!-- FRONT FORK - Caster wheel that follows the differential drive      -->
+  <!-- FRONT FORK - ACTIVELY STEERED wheel (Track A tricycle migration)   -->
+  <!--                                                                    -->
+  <!-- Was: a free 'caster' (continuous swivel) that followed diff-drive. -->
+  <!-- Now: an actively commanded steering axis (revolute steering_joint) -->
+  <!-- driven by ros2_control's tricycle_steering_controller.             -->
+  <!--                                                                    -->
+  <!-- DEST: bglx_ws/src/etrike_description/urdf/components/front_fork.xacro -->
   <!-- ================================================================== -->
   <xacro:property name="front_wheel_radius" value="0.175"/>
   <xacro:property name="front_wheel_width" value="0.05"/>
   <xacro:property name="front_wheel_mass" value="2.0"/>
+  <!-- Steering limit (rad). ~0.6 rad = ~34 deg. With wheelbase 1.33 m this
+       gives minimum turning radius R = L / tan(delta) ~ 1.95 m.
+       Keep in sync with nav2_params planner minimum_turning_radius (>= R)
+       and cmd_vel_limiter.py max_steering_angle. -->
+  <xacro:property name="max_steer" value="0.6"/>
   <xacro:macro name="front_fork" params="parent">
-    <!-- ============================================================== -->
-    <!-- CASTER MOUNT - Allows 360° rotation                            -->
-    <!-- ============================================================== -->
+    <!-- STEERING YOKE (link name kept as caster_mount so gazebo material
+         references in gazebo_config.xacro still resolve). -->
     <link name="caster_mount">
       <inertial>
@@ -19,27 +29,23 @@
       <visual>
         <origin xyz="0 0 0" rpy="0 0 0"/>
-        <geometry>
-          <box size="0.06 0.06 0.04"/>
-        </geometry>
+        <geometry><box size="0.06 0.06 0.04"/></geometry>
         <material name="aluminum"/>
       </visual>
       <collision>
         <origin xyz="0 0 0" rpy="0 0 0"/>
-        <geometry>
-          <box size="0.06 0.06 0.04"/>
-        </geometry>
+        <geometry><box size="0.06 0.06 0.04"/></geometry>
       </collision>
     </link>
-    <!-- Caster swivel joint - free rotation around Z -->
-    <joint name="caster_swivel_joint" type="continuous">
+    <!-- STEERING JOINT: renamed from caster_swivel_joint, changed
+         continuous(free) -> revolute(limited, actively driven). -->
+    <joint name="steering_joint" type="revolute">
       <parent link="frame_head_tube"/>
       <child link="caster_mount"/>
       <origin xyz="0 0 -0.05" rpy="0 0 0"/>
       <axis xyz="0 0 1"/>
-      <dynamics damping="0.01" friction="0.001"/>
+      <limit effort="50.0" velocity="2.0" lower="${-max_steer}" upper="${max_steer}"/>
+      <dynamics damping="0.1" friction="0.05"/>
     </joint>
-    <!-- ============================================================== -->
-    <!-- FORK ASSEMBLY                                                  -->
-    <!-- ============================================================== -->
+    <!-- FORK ASSEMBLY -->
     <link name="steering_link">
       <inertial>
@@ -78,5 +84,4 @@
       </collision>
     </link>
-    <!-- Fork fixed to caster mount (offset creates trailing caster effect) -->
     <joint name="fork_joint" type="fixed">
       <parent link="caster_mount"/>
@@ -84,7 +89,5 @@
       <origin xyz="0 0 0" rpy="0 0 0"/>
     </joint>
-    <!-- ============================================================== -->
-    <!-- FRONT WHEEL                                                    -->
-    <!-- ============================================================== -->
+    <!-- FRONT WHEEL - passive rolling (front is steer-only, not driven) -->
     <link name="front_wheel">
       <inertial>
@@ -95,17 +98,12 @@
       <visual>
         <origin xyz="0 0 0" rpy="${pi/2} 0 0"/>
-        <geometry>
-          <cylinder radius="${front_wheel_radius}" length="${front_wheel_width}"/>
-        </geometry>
+        <geometry><cylinder radius="${front_wheel_radius}" length="${front_wheel_width}"/></geometry>
         <material name="rubber"/>
       </visual>
       <collision>
         <origin xyz="0 0 0" rpy="${pi/2} 0 0"/>
-        <geometry>
-          <cylinder radius="${front_wheel_radius}" length="${front_wheel_width}"/>
-        </geometry>
+        <geometry><cylinder radius="${front_wheel_radius}" length="${front_wheel_width}"/></geometry>
       </collision>
     </link>
-    <!-- Front wheel rotation -->
     <joint name="front_wheel_joint" type="continuous">
       <parent link="steering_link"/>

File: bglx_ws/src/etrike_description/urdf/etrike.urdf.xacro (robot description, xacro)
@@ -2,53 +2,32 @@
 <robot name="bglx_etrike" xmlns:xacro="http://www.ros.org/wiki/xacro">
   <!-- ================================================================== -->
-  <!-- BGLX AUTONOMOUS E-TRIKE                                            -->
-  <!-- Main URDF entry point - includes all components                    -->
+  <!-- BGLX AUTONOMOUS E-TRIKE - Main URDF entry point                    -->
+  <!-- DEST: bglx_ws/src/etrike_description/urdf/etrike.urdf.xacro        -->
+  <!-- Track A change: include the ros2_control / gazebo_ros2_control xacro-->
   <!-- ================================================================== -->
-  <!-- Note: pi is provided by xacro automatically, no need to define it -->
+  <!-- Inertia + material helpers -->
+  <xacro:include filename="$(find etrike_description)/urdf/macros/inertia_macros.xacro"/>
+  <xacro:include filename="$(find etrike_description)/urdf/macros/materials.xacro"/>
+  <!-- Components -->
+  <xacro:include filename="$(find etrike_description)/urdf/components/frame.xacro"/>
+  <xacro:include filename="$(find etrike_description)/urdf/components/front_fork.xacro"/>
+  <xacro:include filename="$(find etrike_description)/urdf/components/control_panel.xacro"/>
+  <xacro:include filename="$(find etrike_description)/urdf/components/battery.xacro"/>
+  <xacro:include filename="$(find etrike_description)/urdf/components/cargo_box.xacro"/>
+  <xacro:include filename="$(find etrike_description)/urdf/components/rear_drive.xacro"/>
+  <xacro:include filename="$(find etrike_description)/urdf/components/sensors.xacro"/>
+  <!-- Gazebo sensor/material config (diff_drive plugin REMOVED here) -->
+  <xacro:include filename="$(find etrike_description)/urdf/gazebo/gazebo_config.xacro"/>
+  <!-- NEW: ros2_control hardware + gazebo_ros2_control plugin -->
+  <xacro:include filename="$(find etrike_description)/urdf/control/etrike_ros2_control.xacro"/>
   <!-- ============================================================== -->
-  <!-- INCLUDE MACROS                                                 -->
+  <!-- INSTANTIATE COMPONENTS (parent links must exist before children)-->
   <!-- ============================================================== -->
-  <!-- Inertia calculation helpers -->
-  <xacro:include filename="$(find etrike_description)/urdf/macros/inertia_macros.xacro"/>
-  <!-- Material/color definitions -->
-  <xacro:include filename="$(find etrike_description)/urdf/macros/materials.xacro"/>
-  <!-- ============================================================== -->
-  <!-- INCLUDE COMPONENTS                                             -->
-  <!-- ============================================================== -->
-  <!-- Main tubular frame -->
-  <xacro:include filename="$(find etrike_description)/urdf/components/frame.xacro"/>
-  <!-- Front fork with steering and wheel -->
-  <xacro:include filename="$(find etrike_description)/urdf/components/front_fork.xacro"/>
-  <!-- Control panel with A-frame and screen -->
-  <xacro:include filename="$(find etrike_description)/urdf/components/control_panel.xacro"/>
-  <!-- Battery enclosure -->
-  <xacro:include filename="$(find etrike_description)/urdf/components/battery.xacro"/>
-  <!-- Cargo box -->
-  <xacro:include filename="$(find etrike_description)/urdf/components/cargo_box.xacro"/>
-  <!-- Rear drive system with hub motors -->
-  <xacro:include filename="$(find etrike_description)/urdf/components/rear_drive.xacro"/>
-  <!-- Sensors (LiDAR, cameras) -->
-  <xacro:include filename="$(find etrike_description)/urdf/components/sensors.xacro"/>
-  <!-- ============================================================== -->
-  <!-- INCLUDE GAZEBO CONFIG (only loaded in simulation)              -->
-  <!-- ============================================================== -->
-  <xacro:include filename="$(find etrike_description)/urdf/gazebo/gazebo_config.xacro"/>
-  <!-- ============================================================== -->
-  <!-- INSTANTIATE COMPONENTS                                         -->
-  <!-- ============================================================== -->
-  <!-- Build order matters! Parent links must exist before children -->
-  <!-- 1. Frame (creates base_link and frame structure) -->
   <xacro:frame parent="base_link"/>
-  <!-- 2. Front fork (attaches to frame_head_tube) -->
   <xacro:front_fork parent="frame_head_tube"/>
-  <!-- 3. Control panel (attaches to frame_main_spine) -->
   <xacro:control_panel parent="frame_main_spine"/>
-  <!-- 4. Battery (attaches to base_link) -->
   <xacro:battery parent="base_link"/>
-  <!-- 5. Cargo box (attaches to base_link) -->
   <xacro:cargo_box parent="base_link"/>
-  <!-- 6. Rear drive (attaches to base_link) -->
   <xacro:rear_drive parent="base_link"/>
-  <!-- 7. Sensors (attaches to sensor_mount_plate and other links) -->
   <xacro:sensors parent="sensor_mount_plate"/>
 </robot>

Commit message: fix(sim): tyre friction 1.5->0.85, positive fork trail, 60 deg steering
Three vehicle-dynamics corrections found by rollover analysis:

- mu 1.5 exceeded the 0.61g stability-triangle threshold, so the trike
  always tipped rather than slid. 0.85 matches rubber on asphalt.
- Front wheel sat 40mm AHEAD of the steering axis: negative trail, so
  steering was actively destabilising. Moved to +60mm, which is normal
  bicycle geometry and eliminates the shimmy.
- Max steer 0.6 -> 1.047 rad (60 deg), cutting minimum turning radius
  from 1.94m to 0.77m and the U-turn corridor from 4.4m to 1.5m.

File: bglx_ws/src/etrike_description/urdf/components/front_fork.xacro (robot description, xacro)
@@ -17,5 +17,5 @@
        Keep in sync with nav2_params planner minimum_turning_radius (>= R)
        and cmd_vel_limiter.py max_steering_angle. -->
-  <xacro:property name="max_steer" value="0.6"/>
+  <xacro:property name="max_steer" value="1.047"/>
   <xacro:macro name="front_fork" params="parent">
     <!-- STEERING YOKE (link name kept as caster_mount so gazebo material
@@ -45,5 +45,5 @@
       <axis xyz="0 0 1"/>
       <limit effort="50.0" velocity="2.0" lower="${-max_steer}" upper="${max_steer}"/>
-      <dynamics damping="0.1" friction="0.05"/>
+      <dynamics damping="3.0" friction="0.5"/>
     </joint>
     <!-- FORK ASSEMBLY -->
@@ -109,5 +109,5 @@
       <parent link="steering_link"/>
       <child link="front_wheel"/>
-      <origin xyz="0.04 0 -0.28" rpy="0 0 0"/>
+      <origin xyz="-0.06 0 -0.28" rpy="0 0 0"/>
       <axis xyz="0 1 0"/>
       <dynamics damping="0.001" friction="0.001"/>

File: bglx_ws/src/etrike_description/urdf/control/etrike_ros2_control.xacro (robot description, xacro)
@@ -24,6 +24,6 @@
     <joint name="steering_joint">
       <command_interface name="position">
-        <param name="min">-0.6</param>
-        <param name="max">0.6</param>
+        <param name="min">-1.047</param>
+        <param name="max">1.047</param>
       </command_interface>
       <state_interface name="position"/>

File: bglx_ws/src/etrike_description/urdf/gazebo/gazebo_config.xacro (robot description, xacro)
@@ -35,6 +35,6 @@
   <gazebo reference="front_wheel">
     <material>Gazebo/FlatBlack</material>
-    <mu1>1.5</mu1>
-    <mu2>1.5</mu2>
+    <mu1>0.85</mu1>
+    <mu2>0.85</mu2>
     <kp>1000000.0</kp>
     <kd>100.0</kd>
@@ -44,6 +44,6 @@
   <gazebo reference="rear_left_wheel">
     <material>Gazebo/FlatBlack</material>
-    <mu1>1.5</mu1>
-    <mu2>1.5</mu2>
+    <mu1>0.85</mu1>
+    <mu2>0.85</mu2>
     <kp>1000000.0</kp>
     <kd>100.0</kd>
@@ -53,6 +53,6 @@
   <gazebo reference="rear_right_wheel">
     <material>Gazebo/FlatBlack</material>
-    <mu1>1.5</mu1>
-    <mu2>1.5</mu2>
+    <mu1>0.85</mu1>
+    <mu2>0.85</mu2>
     <kp>1000000.0</kp>
     <kd>100.0</kd>

Commit message: MPPI controller + 60deg/s steering actuator; suspension fork; straight-reverse routing; SLAM mapping fix
- nav: FollowPath RPP -> MPPI (Ackermann, min_turning_r 0.8) + Reeds-Shepp
  planner for reverse-capable paths; goal/path critic + lookahead tuning
- cmd_vel_limiter: model a 60 deg/s self-locking steering actuator (command
  rate-limit + low-pass) to mitigate MPPI steering wobble without disturbing
  tricycle odometry
- agent: route short reverses (<=5m, no lateral) to a closed-loop straight
  back-up with rear-lidar safety instead of a Nav2 pose goal (removes the
  reverse loop-around); >5m still uses Nav2
- etrike_description: remodel front fork - twin-stanchion suspension look,
  fat tire, disc rotor + caliper (visual only; joints + wheel radius unchanged)
- slam_toolbox: mode localization -> mapping (fresh maps build from scratch)
- controllers: reduce_wheel_speed_until_steering_reached=false

KNOWN TODO (not fixed): reverse/escape safety needs sector-weighted clearance
plus a proper unwedge recovery - agent can still get stuck against walls in
tight spaces. Reverse-clearance experiment reverted (caused a rear-corner
collision).

File: bglx_ws/src/etrike_description/urdf/components/front_fork.xacro (robot description, xacro)
@@ -2,23 +2,20 @@
 <robot xmlns:xacro="http://www.ros.org/wiki/xacro">
   <!-- ================================================================== -->
-  <!-- FRONT FORK - ACTIVELY STEERED wheel (Track A tricycle migration)   -->
+  <!-- FRONT FORK - suspension-fork styling + fat tire + disc brake       -->
   <!--                                                                    -->
-  <!-- Was: a free 'caster' (continuous swivel) that followed diff-drive. -->
-  <!-- Now: an actively commanded steering axis (revolute steering_joint) -->
-  <!-- driven by ros2_control's tricycle_steering_controller.             -->
-  <!--                                                                    -->
+  <!-- VISUAL REMODEL ONLY. Joint names, link names and wheel RADIUS are  -->
+  <!-- unchanged, so tricycle_steering_controller, ros2_control and the   -->
+  <!-- odometry all keep working. Tire is made fatter (width only) and a  -->
+  <!-- disc rotor + caliper + twin-stanchion fork are added for the look. -->
   <!-- DEST: bglx_ws/src/etrike_description/urdf/components/front_fork.xacro -->
   <!-- ================================================================== -->
   <xacro:property name="front_wheel_radius" value="0.175"/>
-  <xacro:property name="front_wheel_width" value="0.05"/>
-  <xacro:property name="front_wheel_mass" value="2.0"/>
-  <!-- Steering limit (rad). ~0.6 rad = ~34 deg. With wheelbase 1.33 m this
-       gives minimum turning radius R = L / tan(delta) ~ 1.95 m.
-       Keep in sync with nav2_params planner minimum_turning_radius (>= R)
-       and cmd_vel_limiter.py max_steering_angle. -->
+  <xacro:property name="front_wheel_width"  value="0.12"/>   <!-- fatter tire (was 0.05) -->
+  <xacro:property name="front_wheel_mass"   value="2.0"/>
+  <!-- Steering limit (rad). ~1.047 rad = 60 deg. Keep in sync with
+       nav2_params minimum_turning_radius and cmd_vel_limiter. -->
   <xacro:property name="max_steer" value="1.047"/>
   <xacro:macro name="front_fork" params="parent">
-    <!-- STEERING YOKE (link name kept as caster_mount so gazebo material
-         references in gazebo_config.xacro still resolve). -->
+    <!-- STEERING YOKE (link name caster_mount kept for joint + material refs) -->
     <link name="caster_mount">
       <inertial>
@@ -29,6 +26,6 @@
       <visual>
         <origin xyz="0 0 0" rpy="0 0 0"/>
-        <geometry><box size="0.06 0.06 0.04"/></geometry>
-        <material name="aluminum"/>
+        <geometry><box size="0.06 0.10 0.05"/></geometry>
+        <material name="fork"/>
       </visual>
       <collision>
@@ -37,6 +34,5 @@
       </collision>
     </link>
-    <!-- STEERING JOINT: renamed from caster_swivel_joint, changed
-         continuous(free) -> revolute(limited, actively driven). -->
+    <!-- STEERING JOINT (unchanged wiring; actively driven revolute) -->
     <joint name="steering_joint" type="revolute">
       <parent link="frame_head_tube"/>
@@ -44,42 +40,65 @@
       <origin xyz="0 0 -0.05" rpy="0 0 0"/>
       <axis xyz="0 0 1"/>
-      <limit effort="50.0" velocity="2.0" lower="${-max_steer}" upper="${max_steer}"/>
-      <dynamics damping="3.0" friction="0.5"/>
+      <limit effort="80.0" velocity="8.0" lower="${-max_steer}" upper="${max_steer}"/>
+      <dynamics damping="1.0" friction="0.1"/>
     </joint>
-    <!-- FORK ASSEMBLY -->
+    <!-- FORK ASSEMBLY: crown + twin upper stanchions + twin lower legs -->
     <link name="steering_link">
       <inertial>
         <mass value="1.0"/>
-        <origin xyz="0 0 -0.12" rpy="0 0 0"/>
-        <xacro:box_inertia m="1.0" x="0.04" y="0.10" z="0.25"/>
+        <origin xyz="0 0 -0.15" rpy="0 0 0"/>
+        <xacro:box_inertia m="1.0" x="0.06" y="0.14" z="0.28"/>
       </inertial>
+      <!-- fork crown (connects legs to steerer) -->
       <visual>
-        <origin xyz="0.02 0 -0.04" rpy="0 0 0"/>
-        <geometry><cylinder radius="0.022" length="0.12"/></geometry>
+        <origin xyz="0.01 0 -0.04" rpy="0 0 0"/>
+        <geometry><box size="0.07 0.15 0.05"/></geometry>
         <material name="fork"/>
       </visual>
+      <!-- steerer stub up into the head tube -->
       <visual>
-        <origin xyz="0.035 0 -0.05" rpy="0 0 0"/>
-        <geometry><box size="0.05 0.13 0.04"/></geometry>
+        <origin xyz="0.0 0 0.01" rpy="0 0 0"/>
+        <geometry><cylinder radius="0.024" length="0.10"/></geometry>
         <material name="fork"/>
       </visual>
+      <!-- LEFT upper stanchion (silver) -->
       <visual>
-        <origin xyz="0.04 0.055 -0.17" rpy="0 0 0"/>
-        <geometry><cylinder radius="0.016" length="0.26"/></geometry>
+        <origin xyz="0.03 0.058 -0.13" rpy="0 0 0"/>
+        <geometry><cylinder radius="0.020" length="0.18"/></geometry>
+        <material name="aluminum"/>
+      </visual>
+      <!-- RIGHT upper stanchion -->
+      <visual>
+        <origin xyz="0.03 -0.058 -0.13" rpy="0 0 0"/>
+        <geometry><cylinder radius="0.020" length="0.18"/></geometry>
+        <material name="aluminum"/>
+      </visual>
+      <!-- LEFT lower leg / slider (fatter, dark) -->
+      <visual>
+        <origin xyz="0.005 0.058 -0.24" rpy="0 0 0"/>
+        <geometry><cylinder radius="0.026" length="0.12"/></geometry>
         <material name="fork"/>
       </visual>
+      <!-- RIGHT lower leg / slider -->
       <visual>
-        <origin xyz="0.04 -0.055 -0.17" rpy="0 0 0"/>
-        <geometry><cylinder radius="0.016" length="0.26"/></geometry>
+        <origin xyz="0.005 -0.058 -0.24" rpy="0 0 0"/>
+        <geometry><cylinder radius="0.026" length="0.12"/></geometry>
         <material name="fork"/>
       </visual>
+      <!-- dropout bridge at the axle -->
       <visual>
-        <origin xyz="0.04 0 -0.28" rpy="1.5708 0 0"/>
-        <geometry><cylinder radius="0.014" length="0.14"/></geometry>
+        <origin xyz="-0.03 0 -0.29" rpy="0 0 0"/>
+        <geometry><box size="0.05 0.14 0.03"/></geometry>
         <material name="fork"/>
       </visual>
+      <!-- brake caliper on left lower leg near rotor top (fixed to fork) -->
+      <visual>
+        <origin xyz="-0.02 0.078 -0.20" rpy="0 0 0"/>
+        <geometry><box size="0.03 0.022 0.06"/></geometry>
+        <material name="hub_motor"/>
+      </visual>
       <collision>
-        <origin xyz="0.035 0 -0.14" rpy="0 0 0"/>
-        <geometry><box size="0.05 0.14 0.26"/></geometry>
+        <origin xyz="0.01 0 -0.15" rpy="0 0 0"/>
+        <geometry><box size="0.06 0.16 0.26"/></geometry>
       </collision>
     </link>
@@ -89,5 +108,5 @@
       <origin xyz="0 0 0" rpy="0 0 0"/>
     </joint>
-    <!-- FRONT WHEEL - passive rolling (front is steer-only, not driven) -->
+    <!-- FRONT WHEEL - passive rolling, FAT tire (radius unchanged) -->
     <link name="front_wheel">
       <inertial>
@@ -113,9 +132,10 @@
       <dynamics damping="0.001" friction="0.001"/>
     </joint>
+    <!-- RIM (widened to match fat tire) -->
     <link name="front_rim">
       <inertial><mass value="0.2"/><origin xyz="0 0 0" rpy="0 0 0"/>
         <inertia ixx="1e-4" ixy="0" ixz="0" iyy="1e-4" iyz="0" izz="1e-4"/></inertial>
       <visual><origin xyz="0 0 0" rpy="${pi/2} 0 0"/>
-        <geometry><cylinder radius="0.11" length="0.052"/></geometry>
+        <geometry><cylinder radius="0.115" length="0.055"/></geometry>
         <material name="aluminum"/></visual>
     </link>
@@ -125,9 +145,10 @@
     </joint>
     <gazebo reference="front_rim"><material>Gazebo/Grey</material></gazebo>
+    <!-- HUB (widened) -->
     <link name="front_hubcap">
       <inertial><mass value="0.05"/><origin xyz="0 0 0" rpy="0 0 0"/>
         <inertia ixx="1e-5" ixy="0" ixz="0" iyy="1e-5" iyz="0" izz="1e-5"/></inertial>
       <visual><origin xyz="0 0 0" rpy="${pi/2} 0 0"/>
-        <geometry><cylinder radius="0.045" length="0.062"/></geometry>
+        <geometry><cylinder radius="0.045" length="0.13"/></geometry>
         <material name="hub_motor"/></visual>
     </link>
@@ -137,4 +158,20 @@
     </joint>
     <gazebo reference="front_hubcap"><material>Gazebo/DarkGrey</material></gazebo>
+    <!-- DISC BRAKE ROTOR (rotates with wheel; brake side = +y) -->
+    <link name="front_disc">
+      <inertial><mass value="0.08"/><origin xyz="0 0 0" rpy="0 0 0"/>
+        <inertia ixx="1e-5" ixy="0" ixz="0" iyy="1e-5" iyz="0" izz="1e-5"/></inertial>
+      <visual><origin xyz="0 0 0" rpy="${pi/2} 0 0"/>
+        <geometry><cylinder radius="0.090" length="0.004"/></geometry>
+        <material name="aluminum"/></visual>
+    </link>
+    <joint name="front_disc_joint" type="fixed">
+      <parent link="front_wheel"/><child link="front_disc"/>
+      <origin xyz="0 0.062 0" rpy="0 0 0"/>
+    </joint>
+    <gazebo reference="front_disc"><material>Gazebo/Grey</material></gazebo>
+    <!-- Gazebo Classic surface colours -->
+    <gazebo reference="front_wheel"><material>Gazebo/FlatBlack</material></gazebo>
+    <gazebo reference="steering_link"><material>Gazebo/FlatBlack</material></gazebo>
   </xacro:macro>
 </robot>
