Commit message: sensors: perimeter depth cams -> ray proximity sensors (1.5Hz -> 15Hz)
Three type=depth cameras saturated Gazebo Classic's render thread at ~1.5Hz. Replaced with type=ray proximity sensors (LaserScan on /etrike/*/scan): negligible render cost, steady 15Hz. Mirrors cheap ToF/ultrasonic sensors the real trike will use.

File: bglx_ws/src/etrike_description/urdf/components/perimeter_sensors.xacro (robot description, xacro)
@@ -1,9 +1,16 @@
 <?xml version="1.0"?>
 <robot xmlns:xacro="http://www.ros.org/wiki/xacro">
-  <!-- Perimeter depth sensing: left / right / rear.
-       Fills the 2D LiDAR's 0.45 m minimum-range blind ring around the body.
-       Mirrors the existing front_depth plugin (libgazebo_ros_camera, /etrike ns).
-       Each cam: aimed outward (yaw) + 15 deg down-pitch, 86 deg HFOV, 0.05-6 m. -->
-  <xacro:macro name="perimeter_depth" params="name parent x y z yaw">
+  <!-- Perimeter PROXIMITY sensing: left / right / rear.
+       Fills the 2D LiDAR's 0.45 m minimum-range blind ring around the body,
+       and catches low obstacles the main LiDAR plane misses (e.g. benches).
+       CHANGED: was 3x type="depth" cameras (full depth image + pointcloud each
+       frame) which saturated Gazebo Classic's single render thread at ~1.5 Hz.
+       Now 3x type="ray" proximity sensors - a small vertical fan of rays, no
+       image, no pointcloud - render cost is negligible so they hit full rate.
+       Mirrors cheap ultrasonic/ToF proximity sensors the real trike will use.
+       Each sensor publishes sensor_msgs/LaserScan on /etrike/<name>/scan,
+       aimed outward (yaw) + ~15 deg down, spanning a narrow vertical wedge so
+       it sees the ground-plane blind zone without the full LiDAR cost. -->
+  <xacro:macro name="perimeter_prox" params="name parent x y z yaw">
     <link name="${name}_link">
       <visual><origin xyz="0 0 0" rpy="0 0 0"/>
@@ -18,27 +25,38 @@
       <origin xyz="${x} ${y} ${z}" rpy="0 0.26 ${yaw}"/>
     </joint>
-    <!-- optical frame: same convention as depth_camera_optical -->
-    <link name="${name}_optical"/>
-    <joint name="${name}_optical_joint" type="fixed">
-      <parent link="${name}_link"/><child link="${name}_optical"/>
-      <origin xyz="0 0 0" rpy="-1.5708 0 -1.5708"/>
-    </joint>
     <gazebo reference="${name}_link">
       <material>Gazebo/Black</material>
-      <sensor name="${name}" type="depth">
+      <sensor name="${name}" type="ray">
         <always_on>true</always_on>
-        <update_rate>10</update_rate>
+        <update_rate>15</update_rate>
         <visualize>false</visualize>
-        <camera name="${name}">
-          <horizontal_fov>1.50</horizontal_fov>
-          <image><width>240</width><height>180</height><format>R8G8B8</format></image>
-          <clip><near>0.05</near><far>6.0</far></clip>
-        </camera>
-        <plugin filename="libgazebo_ros_camera.so" name="${name}_controller">
-          <ros><namespace>/etrike</namespace></ros>
-          <camera_name>${name}</camera_name>
-          <frame_name>${name}_optical</frame_name>
-          <min_depth>0.05</min_depth>
-          <max_depth>6.0</max_depth>
+        <ray>
+          <scan>
+            <horizontal>
+              <samples>15</samples>
+              <resolution>1</resolution>
+              <min_angle>-0.35</min_angle>
+              <max_angle>0.35</max_angle>
+            </horizontal>
+            <vertical>
+              <samples>5</samples>
+              <resolution>1</resolution>
+              <min_angle>-0.20</min_angle>
+              <max_angle>0.20</max_angle>
+            </vertical>
+          </scan>
+          <range>
+            <min>0.05</min>
+            <max>4.0</max>
+            <resolution>0.01</resolution>
+          </range>
+        </ray>
+        <plugin filename="libgazebo_ros_ray_sensor.so" name="${name}_controller">
+          <ros>
+            <namespace>/etrike</namespace>
+            <remapping>~/out:=${name}/scan</remapping>
+          </ros>
+          <output_type>sensor_msgs/LaserScan</output_type>
+          <frame_name>${name}_link</frame_name>
         </plugin>
       </sensor>
@@ -46,8 +64,8 @@
   </xacro:macro>
   <xacro:macro name="perimeter_sensors" params="parent">
-    <!--                     name         parent      x      y      z     yaw    -->
-    <xacro:perimeter_depth name="left_depth"  parent="${parent}" x="0.45"  y="0.28"  z="0.45" yaw="1.5708"/>
-    <xacro:perimeter_depth name="right_depth" parent="${parent}" x="0.45"  y="-0.28" z="0.45" yaw="-1.5708"/>
-    <xacro:perimeter_depth name="rear_depth"  parent="${parent}" x="-0.10" y="0.0"   z="0.45" yaw="3.14159"/>
+    <!--                    name         parent      x      y      z     yaw    -->
+    <xacro:perimeter_prox name="left_depth"  parent="${parent}" x="0.45"  y="0.28"  z="0.45" yaw="1.5708"/>
+    <xacro:perimeter_prox name="right_depth" parent="${parent}" x="0.45"  y="-0.28" z="0.45" yaw="-1.5708"/>
+    <xacro:perimeter_prox name="rear_depth"  parent="${parent}" x="-0.10" y="0.0"   z="0.45" yaw="3.14159"/>
   </xacro:macro>
 </robot>
