Commit message: sensors: front lidar at 0.30m, perimeter proximity rays, rviz costmap views
Adds a low-mounted forward lidar (front_lidar_link at x=1.05, z=0.35, 15Hz,
5m range, +/-120 deg) because the main scan plane sits at 0.92m and looks
straight over anything shorter: a 0.6m bench and a 0.9m urn are both
invisible to it. Perimeter rays cover left, right and rear at short range.

Verified the low lidar sees the urn: 47 finite returns, all within 30 deg of
straight ahead, closest around 3m. The sensing gap is closed; what remains is
downstream of it.

File: bglx_ws/src/etrike_description/urdf/components/control_panel.xacro (robot description, xacro)
@@ -90,5 +90,5 @@
       <parent link="aframe_leg_left"/>
       <child link="aframe_crossbar"/>
-      <origin xyz="0.05 -0.06 0.30" rpy="0 0 0"/>
+      <origin xyz="0.05 -0.06 0.30" rpy="0 0 ${-10*pi/180}"/>
     </joint>
     <!-- ============================================================== -->

File: bglx_ws/src/etrike_description/urdf/components/frame.xacro (robot description, xacro)
@@ -32,5 +32,5 @@
       <parent link="base_link"/>
       <child link="base_footprint"/>
-      <origin xyz="0 0 0" rpy="0 0 0"/>
+      <origin xyz="0 0 -0.053" rpy="0 0 0"/>
     </joint>
     <!-- ============================================================== -->

File: bglx_ws/src/etrike_description/urdf/components/perimeter_sensors.xacro (robot description, xacro)
@@ -68,4 +68,26 @@
     <xacro:perimeter_prox name="right_depth" parent="${parent}" x="0.45"  y="-0.28" z="0.45" yaw="-1.5708"/>
     <xacro:perimeter_prox name="rear_depth"  parent="${parent}" x="-0.10" y="0.0"   z="0.45" yaw="3.14159"/>
+      <link name="front_lidar_link">
+      <inertial>
+        <mass value="0.25"/>
+        <origin xyz="0 0 0" rpy="0 0 0"/>
+        <inertia ixx="0.000152" ixy="0" ixz="0"
+                 iyy="0.000152" iyz="0" izz="0.0002"/>
+      </inertial>
+      <visual>
+        <origin xyz="0 0 0" rpy="0 0 0"/>
+        <geometry><cylinder radius="0.04" length="0.05"/></geometry>
+        <material name="lidar"/>
+      </visual>
+      <collision>
+        <origin xyz="0 0 0" rpy="0 0 0"/>
+        <geometry><cylinder radius="0.04" length="0.05"/></geometry>
+      </collision>
+    </link>
+    <joint name="front_lidar_joint" type="fixed">
+      <parent link="${parent}"/>
+      <child link="front_lidar_link"/>
+      <origin xyz="1.05 0 0.30" rpy="0 0 0"/>
+    </joint>
   </xacro:macro>
 </robot>

File: bglx_ws/src/etrike_description/urdf/components/sensors.xacro (robot description, xacro)
@@ -242,30 +242,4 @@
     <!-- GROUND CAMERA - Downward facing for close obstacle detection   -->
     <!-- ============================================================== -->
-    <link name="camera_ground">
-      <inertial>
-        <mass value="0.05"/>
-        <origin xyz="0 0 0" rpy="0 0 0"/>
-        <xacro:box_inertia m="0.05" x="0.02" y="0.02" z="0.02"/>
-      </inertial>
-      <visual>
-        <origin xyz="0 0 0" rpy="0 0 0"/>
-        <geometry>
-          <box size="0.02 0.02 0.02"/>
-        </geometry>
-        <material name="carbon_fiber"/>
-      </visual>
-      <collision>
-        <origin xyz="0 0 0" rpy="0 0 0"/>
-        <geometry>
-          <box size="0.02 0.02 0.02"/>
-        </geometry>
-      </collision>
-    </link>
-    <joint name="camera_ground_joint" type="fixed">
-      <parent link="cargo_box"/>
-      <child link="camera_ground"/>
-      <!-- Under cargo box front, angled down 45° -->
-      <origin xyz="0.20 0 -0.18" rpy="0 0.7 0"/>
-    </joint>
   </xacro:macro>
 </robot>

File: bglx_ws/src/etrike_description/urdf/gazebo/gazebo_config.xacro (robot description, xacro)
@@ -29,5 +29,4 @@
   <gazebo reference="camera_rear_right"><material>Gazebo/Black</material></gazebo>
   <gazebo reference="camera_rear_main"><material>Gazebo/Black</material></gazebo>
-  <gazebo reference="camera_ground"><material>Gazebo/Black</material></gazebo>
   <!-- ============================================================== -->
   <!-- WHEEL FRICTION                                                 -->
@@ -161,32 +160,4 @@
   <!-- GROUND CAMERA - Close obstacle detection                       -->
   <!-- ============================================================== -->
-  <gazebo reference="camera_ground">
-    <sensor name="camera_ground" type="camera">
-      <always_on>true</always_on>
-      <visualize>true</visualize>
-      <update_rate>15</update_rate>
-      <camera name="ground">
-        <horizontal_fov>1.2</horizontal_fov>
-        <image>
-          <width>320</width>
-          <height>240</height>
-          <format>R8G8B8</format>
-        </image>
-        <clip>
-          <near>0.05</near>
-          <far>5</far>
-        </clip>
-      </camera>
-      <plugin name="camera_ground_controller" filename="libgazebo_ros_camera.so">
-        <ros>
-          <namespace>/etrike</namespace>
-          <remapping>image_raw:=camera/ground/image_raw</remapping>
-          <remapping>camera_info:=camera/ground/camera_info</remapping>
-        </ros>
-        <camera_name>ground</camera_name>
-        <frame_name>camera_ground</frame_name>
-      </plugin>
-    </sensor>
-  </gazebo>
   <!-- ============================================================== -->
   <!-- IMU SENSOR                                                     -->
@@ -282,3 +253,38 @@
     </sensor>
   </gazebo>
+  <gazebo reference="front_lidar_link">
+    <sensor name="front_lidar" type="ray">
+      <always_on>true</always_on>
+      <visualize>true</visualize>
+      <update_rate>15</update_rate>
+      <ray>
+        <scan>
+          <horizontal>
+            <samples>360</samples>
+            <resolution>1</resolution>
+            <min_angle>-2.0944</min_angle>
+            <max_angle>2.0944</max_angle>
+          </horizontal>
+        </scan>
+        <range>
+          <min>0.15</min>
+          <max>5.0</max>
+          <resolution>0.01</resolution>
+        </range>
+        <noise>
+          <type>gaussian</type>
+          <mean>0.0</mean>
+          <stddev>0.01</stddev>
+        </noise>
+      </ray>
+      <plugin name="front_scan" filename="libgazebo_ros_ray_sensor.so">
+        <ros>
+          <namespace>/etrike</namespace>
+          <remapping>~/out:=front_scan</remapping>
+        </ros>
+        <output_type>sensor_msgs/LaserScan</output_type>
+        <frame_name>front_lidar_link</frame_name>
+      </plugin>
+    </sensor>
+  </gazebo>
 </robot>
