Commit message: checkpoint: preserve rover description and Gazebo integration changes

File: bglx_ws/src/bglx_rover_description/urdf/bglx_rover.urdf.xacro (robot description, xacro)
@@ -54,4 +54,5 @@
       <origin xyz="0 ${reflect*wheel_sep/2} ${wheel_radius - base_h}"/>
       <axis xyz="0 1 0"/>
+      <limit effort="10.0" velocity="20.0"/>
       <dynamics damping="0.02" friction="0.0"/>
     </joint>

File: bglx_ws/src/bglx_rover_description/urdf/control/rover_ros2_control.xacro (robot description, xacro)
@@ -26,4 +26,7 @@
   <gazebo>
     <plugin filename="libgazebo_ros2_control.so" name="gazebo_ros2_control">
+      <ros>
+        <namespace>/rover</namespace>
+      </ros>
       <parameters>$(arg controllers_file)</parameters>
       <robot_param>robot_description</robot_param>

File: bglx_ws/src/bglx_rover_description/urdf/gazebo/gazebo_config.xacro (robot description, xacro)
@@ -21,13 +21,13 @@
   <gazebo reference="caster_front">
     <material>Gazebo/Grey</material>
-    <mu1>0.0</mu1><mu2>0.0</mu2>
+    <mu1>0.1</mu1><mu2>0.1</mu2>
     <kp>1000000.0</kp><kd>100.0</kd>
-    <minDepth>0.001</minDepth>
+    <minDepth>0.001</minDepth><maxVel>0.0</maxVel>
   </gazebo>
   <gazebo reference="caster_rear">
     <material>Gazebo/Grey</material>
-    <mu1>0.0</mu1><mu2>0.0</mu2>
+    <mu1>0.1</mu1><mu2>0.1</mu2>
     <kp>1000000.0</kp><kd>100.0</kd>
-    <minDepth>0.001</minDepth>
+    <minDepth>0.001</minDepth><maxVel>0.0</maxVel>
   </gazebo>
   <gazebo reference="lidar_link">
