Commit message: checkpoint: integrate new trike body and scan filtering fixes
Preserve current trike description, navigation and agent integration.
Enable LiDAR clearing and target rear-wheel self-returns in the front filter.

Simulation evidence:
- Reverse U-turn succeeded without repeated steering centring.
- Forward-turn probe reported zero floor-stop, scan-evidence and collision warnings.
- Forward U-turn remains unresolved: steering commands changed direction;
  trial cancelled at 40 seconds.

Rear-wheel filtering margin and braking/latency values remain experimental.
Runtime trial overrides are not automatically persisted by this commit.

File: bglx_ws/src/etrike_description/urdf/etrike.urdf.xacro (robot description, xacro)
@@ -1,35 +1,1164 @@
-<?xml version="1.0"?>
-<robot name="bglx_etrike" xmlns:xacro="http://www.ros.org/wiki/xacro">
-  <!-- ================================================================== -->
-  <!-- BGLX AUTONOMOUS E-TRIKE - Main URDF entry point                    -->
-  <!-- DEST: bglx_ws/src/etrike_description/urdf/etrike.urdf.xacro        -->
-  <!-- Track A change: include the ros2_control / gazebo_ros2_control xacro-->
-  <!-- ================================================================== -->
-  <!-- Inertia + material helpers -->
-  <xacro:include filename="$(find etrike_description)/urdf/macros/inertia_macros.xacro"/>
-  <xacro:include filename="$(find etrike_description)/urdf/macros/materials.xacro"/>
-  <!-- Components -->
-  <xacro:include filename="$(find etrike_description)/urdf/components/frame.xacro"/>
-  <xacro:include filename="$(find etrike_description)/urdf/components/front_fork.xacro"/>
-  <xacro:include filename="$(find etrike_description)/urdf/components/control_panel.xacro"/>
-  <xacro:include filename="$(find etrike_description)/urdf/components/battery.xacro"/>
-  <xacro:include filename="$(find etrike_description)/urdf/components/cargo_box.xacro"/>
-  <xacro:include filename="$(find etrike_description)/urdf/components/rear_drive.xacro"/>
-  <xacro:include filename="$(find etrike_description)/urdf/components/sensors.xacro"/>
-  <!-- Gazebo sensor/material config (diff_drive plugin REMOVED here) -->
-  <xacro:include filename="$(find etrike_description)/urdf/gazebo/gazebo_config.xacro"/>
-  <!-- NEW: ros2_control hardware + gazebo_ros2_control plugin -->
-  <xacro:include filename="$(find etrike_description)/urdf/control/etrike_ros2_control.xacro"/>
-  <xacro:include filename="$(find etrike_description)/urdf/components/perimeter_sensors.xacro"/>
-  <!-- ============================================================== -->
-  <!-- INSTANTIATE COMPONENTS (parent links must exist before children)-->
-  <!-- ============================================================== -->
-  <xacro:frame parent="base_link"/>
-  <xacro:front_fork parent="frame_head_tube"/>
-  <xacro:control_panel parent="frame_main_spine"/>
-  <xacro:battery parent="base_link"/>
-  <xacro:cargo_box parent="base_link"/>
-  <xacro:rear_drive parent="base_link"/>
-  <xacro:sensors parent="sensor_mount_plate"/>
-  <xacro:perimeter_sensors parent="base_link"/>
+<robot xmlns:xacro="http://www.ros.org/wiki/xacro" name="bglx_production_concept">
+  <xacro:arg name="controllers_file" default="$(find etrike_description)/config/controllers.yaml" /><material name="concept_mount">
+    <color rgba="0.22 0.26 0.23 1" />
+  </material>
+  <link name="base_link">
+    <inertial>
+      <origin rpy="0 0 0" xyz="0.4568493151 0 0.452739726" />
+      <mass value="29.2" />
+      <inertia ixx="2.501097489" ixy="0" ixz="0.8218479452" iyy="4.096344292" iyz="0" izz="2.346680137" />
+    </inertial>
+    <collision name="lower_chassis">
+      <origin rpy="0 0 0" xyz="0.48 0 0.2225" />
+      <geometry>
+        <box size="1.04 0.38 0.095" />
+      </geometry>
+    </collision>
+    <collision name="battery">
+      <origin rpy="0 0 0" xyz="0.55 0 0.335" />
+      <geometry>
+        <box size="0.58 0.32 0.2" />
+      </geometry>
+    </collision>
+    <collision name="cargo_shell">
+      <origin rpy="0 0 0" xyz="0.18 0 0.882" />
+      <geometry>
+        <box size="0.7 0.61 0.58" />
+      </geometry>
+    </collision>
+    <collision name="cargo_support">
+      <origin rpy="0 0 0" xyz="0.13 0 0.44" />
+      <geometry>
+        <box size="0.36 0.47 0.32" />
+      </geometry>
+    </collision>
+    <collision name="display">
+      <origin rpy="0 -0.3 0" xyz="0.97 0 0.785" />
+      <geometry>
+        <box size="0.06 0.225 0.375" />
+      </geometry>
+    </collision>
+    <collision name="head_bearing_support">
+      <origin rpy="0 0 0" xyz="1.08 0 0.64" />
+      <geometry>
+        <box size="0.28 0.065 0.03" />
+      </geometry>
+    </collision>
+    <visual name="head_bearing_support">
+      <origin rpy="0 0 0" xyz="1.08 0 0.64" />
+      <geometry>
+        <box size="0.28 0.065 0.03" />
+      </geometry>
+      <material name="bglx_aluminum">
+        <color rgba="0.68 0.71 0.68 1.0" />
+      </material>
+    </visual>
+    <collision name="sensor_mast">
+      <origin rpy="0 0 0" xyz="0.42 0 1.243" />
+      <geometry>
+        <box size="0.23 0.34 0.142" />
+      </geometry>
+    </collision>
+    <collision name="terrain_camera_mount">
+      <origin rpy="0 0 0" xyz="1.005 0 0.855" />
+      <geometry>
+        <box size="0.095 0.07 0.025" />
+      </geometry>
+    </collision>
+    <visual name="terrain_camera_mount">
+      <origin rpy="0 0 0" xyz="1.005 0 0.855" />
+      <geometry>
+        <box size="0.095 0.07 0.025" />
+      </geometry>
+      <material name="bglx_aluminum">
+        <color rgba="0.68 0.71 0.68 1.0" />
+      </material>
+    </visual>
+    <visual name="bglx_color_body_0">
+      <origin rpy="0 0 0" xyz="0 0 0" />
+      <geometry>
+        <mesh filename="package://etrike_description/meshes/concept_color/body_0.stl" scale="1 1 1" />
+      </geometry>
+      <material name="bglx_color_body_0">
+        <color rgba="0.627451 0.666667 0.635294 1.0" />
+      </material>
+    </visual>
+    <visual name="bglx_color_body_1">
+      <origin rpy="0 0 0" xyz="0 0 0" />
+      <geometry>
+        <mesh filename="package://etrike_description/meshes/concept_color/body_1.stl" scale="1 1 1" />
+      </geometry>
+      <material name="bglx_color_body_1">
+        <color rgba="0.466667 0.494118 0.470588 1.0" />
+      </material>
+    </visual>
+    <visual name="bglx_color_body_2">
+      <origin rpy="0 0 0" xyz="0 0 0" />
+      <geometry>
+        <mesh filename="package://etrike_description/meshes/concept_color/body_2.stl" scale="1 1 1" />
+      </geometry>
+      <material name="bglx_color_body_2">
+        <color rgba="0.737255 0.772549 0.737255 1.0" />
+      </material>
+    </visual>
+    <visual name="bglx_color_body_3">
+      <origin rpy="0 0 0" xyz="0 0 0" />
+      <geometry>
+        <mesh filename="package://etrike_description/meshes/concept_color/body_3.stl" scale="1 1 1" />
+      </geometry>
+      <material name="bglx_color_body_3">
+        <color rgba="0.223529 0.262745 0.231373 1.0" />
+      </material>
+    </visual>
+    <visual name="bglx_color_body_4">
+      <origin rpy="0 0 0" xyz="0 0 0" />
+      <geometry>
+        <mesh filename="package://etrike_description/meshes/concept_color/body_4.stl" scale="1 1 1" />
+      </geometry>
+      <material name="bglx_color_body_4">
+        <color rgba="0.141176 0.160784 0.145098 1.0" />
+      </material>
+    </visual>
+    <visual name="bglx_color_body_5">
+      <origin rpy="0 0 0" xyz="0 0 0" />
+      <geometry>
+        <mesh filename="package://etrike_description/meshes/concept_color/body_5.stl" scale="1 1 1" />
+      </geometry>
+      <material name="bglx_color_body_5">
+        <color rgba="0.062745 0.090196 0.07451 1.0" />
+      </material>
+    </visual>
+    <visual name="bglx_color_body_6">
+      <origin rpy="0 0 0" xyz="0 0 0" />
+      <geometry>
+        <mesh filename="package://etrike_description/meshes/concept_color/body_6.stl" scale="1 1 1" />
+      </geometry>
+      <material name="bglx_color_body_6">
+        <color rgba="0.043137 0.094118 0.066667 1.0" />
+      </material>
+    </visual>
+    <visual name="bglx_color_body_7">
+      <origin rpy="0 0 0" xyz="0 0 0" />
+      <geometry>
+        <mesh filename="package://etrike_description/meshes/concept_color/body_7.stl" scale="1 1 1" />
+      </geometry>
+      <material name="bglx_color_body_7">
+        <color rgba="0.329412 0.72549 0.482353 1.0" />
+      </material>
+    </visual>
+    <visual name="bglx_color_body_8">
+      <origin rpy="0 0 0" xyz="0 0 0" />
+      <geometry>
+        <mesh filename="package://etrike_description/meshes/concept_color/body_8.stl" scale="1 1 1" />
+      </geometry>
+      <material name="bglx_color_body_8">
+        <color rgba="0.207843 0.227451 0.215686 1.0" />
+      </material>
+    </visual>
+    <visual name="bglx_color_body_9">
+      <origin rpy="0 0 0" xyz="0 0 0" />
+      <geometry>
+        <mesh filename="package://etrike_description/meshes/concept_color/body_9.stl" scale="1 1 1" />
+      </geometry>
+      <material name="bglx_color_body_9">
+        <color rgba="0.188235 0.207843 0.196078 1.0" />
+      </material>
+    </visual>
+    <visual name="bglx_color_body_10">
+      <origin rpy="0 0 0" xyz="0 0 0" />
+      <geometry>
+        <mesh filename="package://etrike_description/meshes/concept_color/body_10.stl" scale="1 1 1" />
+      </geometry>
+      <material name="bglx_color_body_10">
+        <color rgba="0.031373 0.14902 0.133333 1.0" />
+      </material>
+    </visual>
+  </link>
+  <link name="base_footprint" />
+  <joint name="base_footprint_joint" type="fixed">
+    <parent link="base_link" />
+    <child link="base_footprint" />
+    <origin rpy="0 0 0" xyz="0 0 0" />
+  </joint>
+  <link name="caster_mount">
+    <inertial>
+      <origin rpy="0 0 0" xyz="-0.025 0 -0.19" />
+      <mass value="3" />
+      <inertia ixx="0.052" ixy="0" ixz="0" iyy="0.048" iyz="0" izz="0.015" />
+    </inertial>
+    <collision name="fork_-1">
+      <origin rpy="0 -0.15 0" xyz="-0.025 -0.076 -0.215" />
+      <geometry>
+        <box size="0.047 0.047 0.3" />
+      </geometry>
+    </collision>
+    <collision name="fork_1">
+      <origin rpy="0 -0.15 0" xyz="-0.025 0.076 -0.215" />
+      <geometry>
+        <box size="0.047 0.047 0.3" />
+      </geometry>
+    </collision>
+    <collision name="fork_crown">
+      <origin rpy="0 0 0" xyz="-0.07 0 -0.075" />
+      <geometry>
+        <box size="0.09 0.2 0.04" />
+      </geometry>
+    </collision>
+    <collision name="offset_fork_crown">
+      <origin rpy="0 0 0" xyz="-0.035 0 -0.075" />
+      <geometry>
+        <box size="0.15 0.07 0.038" />
+      </geometry>
+    </collision>
+    <visual name="offset_fork_crown">
+      <origin rpy="0 0 0" xyz="-0.035 0 -0.075" />
+      <geometry>
+        <box size="0.15 0.07 0.038" />
+      </geometry>
+      <material name="bglx_aluminum">
+        <color rgba="0.68 0.71 0.68 1.0" />
+      </material>
+    </visual>
+    <collision name="mudguard_0">
+      <origin rpy="0 1.216818957 0" xyz="0.2814004365 0 -0.2610106046" />
+      <geometry>
+        <box size="0.101 0.12 0.016" />
+      </geometry>
+    </collision>
+    <collision name="mudguard_1">
+      <origin rpy="0 0.9088642179 0" xyz="0.2366418447 0 -0.1806073827" />
+      <geometry>
+        <box size="0.101 0.12 0.016" />
+      </geometry>
+    </collision>
+    <collision name="mudguard_2">
+      <origin rpy="0 0.6009094786 0" xyz="0.1696178594 0 -0.117553477" />
+      <geometry>
+        <box size="0.101 0.12 0.016" />
+      </geometry>
+    </collision>
+    <collision name="mudguard_3">
+      <origin rpy="0 0.2929547393 0" xyz="0.08663470007 0 -0.07778156615" />
+      <geometry>
+        <box size="0.101 0.12 0.016" />
+      </geometry>
+    </collision>
+    <collision name="mudguard_4">
+      <origin rpy="0 -0.015 0" xyz="-0.004499831252 0 -0.06503374937" />
+      <geometry>
+        <box size="0.101 0.12 0.016" />
+      </geometry>
+    </collision>
+    <collision name="mudguard_5">
+      <origin rpy="0 -0.3229547393 0" xyz="-0.09521097797 0 -0.08050945591" />
+      <geometry>
+        <box size="0.101 0.12 0.016" />
+      </geometry>
+    </collision>
+    <collision name="mudguard_6">
+      <origin rpy="0 -0.6309094786 0" xyz="-0.1769638194 0 -0.1227525921" />
+      <geometry>
+        <box size="0.101 0.12 0.016" />
+      </geometry>
+    </collision>
+    <collision name="mudguard_7">
+      <origin rpy="0 -0.9388642179 0" xyz="-0.2420663127 0 -0.1877885437" />
+      <geometry>
+        <box size="0.101 0.12 0.016" />
+      </geometry>
+    </collision>
+    <collision name="mudguard_8">
+      <origin rpy="0 -1.246818957 0" xyz="-0.2843930297 0 -0.2694981432" />
+      <geometry>
+        <box size="0.101 0.12 0.016" />
+      </geometry>
+    </collision>
+    <collision name="axle_sensor">
+      <origin rpy="0 0 0" xyz="0.035 0.145 -0.34" />
+      <geometry>
+        <box size="0.08 0.075 0.065" />
+      </geometry>
+    </collision>
+    <visual name="bglx_color_steering_0">
+      <origin rpy="0 0 0" xyz="-0.07 0 0" />
+      <geometry>
+        <mesh filename="package://etrike_description/meshes/concept_color/steering_0.stl" scale="1 1 1" />
+      </geometry>
+      <material name="bglx_color_steering_0">
+        <color rgba="0.627451 0.666667 0.635294 1.0" />
+      </material>
+    </visual>
+    <visual name="bglx_color_steering_1">
+      <origin rpy="0 0 0" xyz="-0.07 0 0" />
+      <geometry>
+        <mesh filename="package://etrike_description/meshes/concept_color/steering_1.stl" scale="1 1 1" />
+      </geometry>
+      <material name="bglx_color_steering_1">
+        <color rgba="0.223529 0.262745 0.231373 1.0" />
+      </material>
+    </visual>
+    <visual name="bglx_color_steering_2">
+      <origin rpy="0 0 0" xyz="-0.07 0 0" />
+      <geometry>
+        <mesh filename="package://etrike_description/meshes/concept_color/steering_2.stl" scale="1 1 1" />
+      </geometry>
+      <material name="bglx_color_steering_2">
+        <color rgba="0.737255 0.772549 0.737255 1.0" />
+      </material>
+    </visual>
+    <visual name="bglx_color_steering_3">
+      <origin rpy="0 0 0" xyz="-0.07 0 0" />
+      <geometry>
+        <mesh filename="package://etrike_description/meshes/concept_color/steering_3.stl" scale="1 1 1" />
+      </geometry>
+      <material name="bglx_color_steering_3">
+        <color rgba="0.062745 0.090196 0.07451 1.0" />
+      </material>
+    </visual>
+    <visual name="bglx_color_steering_4">
+      <origin rpy="0 0 0" xyz="-0.07 0 0" />
+      <geometry>
+        <mesh filename="package://etrike_description/meshes/concept_color/steering_4.stl" scale="1 1 1" />
+      </geometry>
+      <material name="bglx_color_steering_4">
+        <color rgba="0.141176 0.160784 0.145098 1.0" />
+      </material>
+    </visual>
+    <visual name="bglx_color_steering_5">
+      <origin rpy="0 0 0" xyz="-0.07 0 0" />
+      <geometry>
+        <mesh filename="package://etrike_description/meshes/concept_color/steering_5.stl" scale="1 1 1" />
+      </geometry>
+      <material name="bglx_color_steering_5">
+        <color rgba="0.031373 0.14902 0.133333 1.0" />
+      </material>
+    </visual>
+    <visual name="bglx_color_steering_6">
+      <origin rpy="0 0 0" xyz="-0.07 0 0" />
+      <geometry>
+        <mesh filename="package://etrike_description/meshes/concept_color/steering_6.stl" scale="1 1 1" />
+      </geometry>
+      <material name="bglx_color_steering_6">
+        <color rgba="0.203922 0.47451 0.352941 1.0" />
+      </material>
+    </visual>
+  <visual name="clean_front_bracket_0"><origin xyz="0.29500000000000004 0.0 -0.20500000000000002" rpy="0 2.356194490192345 0" /><geometry><cylinder radius="0.009" length="0.09899494936611665" /></geometry><material name="clean_sensor_bracket"><color rgba="0.12 0.14 0.13 1" /></material></visual><collision name="clean_front_bracket_0"><origin xyz="0.29500000000000004 0.0 -0.20500000000000002" rpy="0 2.356194490192345 0" /><geometry><cylinder radius="0.009" length="0.09899494936611665" /></geometry></collision><visual name="clean_front_bracket_1"><origin xyz="0.34099999999999997 0.0 -0.27" rpy="0 2.790147859586242 0" /><geometry><cylinder radius="0.009" length="0.06390618123468182" /></geometry><material name="clean_sensor_bracket"><color rgba="0.12 0.14 0.13 1" /></material></visual><collision name="clean_front_bracket_1"><origin xyz="0.34099999999999997 0.0 -0.27" rpy="0 2.790147859586242 0" /><geometry><cylinder radius="0.009" length="0.06390618123468182" /></geometry></collision></link>
+  <joint name="steering_joint" type="revolute">
+    <parent link="base_link" />
+    <child link="caster_mount" />
+    <origin rpy="0 0 0" xyz="1.2 0 0.64" />
+    <axis xyz="0 0 1" />
+    <limit effort="80" lower="-1.047" upper="1.047" velocity="1.047" />
+    <dynamics damping=".4" friction=".02" />
+  </joint>
+  <link name="front_wheel">
+    <inertial>
+      <origin rpy="0 0 0" xyz="0 0 0" />
+      <mass value="2" />
+      <inertia ixx="0.0402125" ixy="0" ixz="0" iyy="0.075625" iyz="0" izz="0.0402125" />
+    </inertial>
+    <collision name="front_wheel_contact">
+      <origin rpy="1.570796327 0 0" xyz="0 0 0" />
+      <geometry>
+        <cylinder length="0.12" radius=".275" />
+      </geometry>
+    </collision>
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