Commit message: feat(sim): checkpoint Delivery C arrival and floor extension

File: bglx_ws/src/etrike_description/urdf/etrike.urdf.xacro (robot description, xacro)
@@ -1,52 +1,53 @@
-<robot xmlns:xacro="http://www.ros.org/wiki/xacro" name="bglx_production_concept">
-  <xacro:arg name="controllers_file" default="$(find etrike_description)/config/controllers.yaml" /><material name="concept_mount">
+<robot xmlns:xacro="http://www.ros.org/wiki/xacro" name="bglx_prototype_proxy">
+  <xacro:arg name="controllers_file" default="$(find etrike_description)/config/controllers.yaml" />
+  <material name="concept_mount">
     <color rgba="0.22 0.26 0.23 1" />
   </material>
   <link name="base_link">
     <inertial>
-      <origin rpy="0 0 0" xyz="0.4568493151 0 0.452739726" />
-      <mass value="29.2" />
-      <inertia ixx="2.501097489" ixy="0" ixz="0.8218479452" iyy="4.096344292" iyz="0" izz="2.346680137" />
+      <origin rpy="0 0 0" xyz="0.342636986325 0 0.307739726" />
+      <mass value="28.52258852258852" />
+      <inertia ixx="2.2081942096410256" ixy="0.0" ixz="0.6020864067399267" iyy="3.159021024542125" iyz="0.0" izz="1.215067108175824" />
     </inertial>
     <collision name="lower_chassis">
-      <origin rpy="0 0 0" xyz="0.48 0 0.2225" />
-      <geometry>
-        <box size="1.04 0.38 0.095" />
+      <origin rpy="0 0 0" xyz="0.36 0 0.0775" />
+      <geometry>
+        <box size="0.78 0.228 0.095" />
       </geometry>
     </collision>
     <collision name="battery">
-      <origin rpy="0 0 0" xyz="0.55 0 0.335" />
-      <geometry>
-        <box size="0.58 0.32 0.2" />
+      <origin rpy="0 0 0" xyz="0.4125 0 0.19" />
+      <geometry>
+        <box size="0.435 0.192 0.2" />
       </geometry>
     </collision>
     <collision name="cargo_shell">
-      <origin rpy="0 0 0" xyz="0.18 0 0.882" />
-      <geometry>
-        <box size="0.7 0.61 0.58" />
+      <origin rpy="0 0 0" xyz="0.135 0 0.737" />
+      <geometry>
+        <box size="0.525 0.366 0.58" />
       </geometry>
     </collision>
     <collision name="cargo_support">
-      <origin rpy="0 0 0" xyz="0.13 0 0.44" />
-      <geometry>
-        <box size="0.36 0.47 0.32" />
+      <origin rpy="0 0 0" xyz="0.0975 0 0.295" />
+      <geometry>
+        <box size="0.27 0.282 0.32" />
       </geometry>
     </collision>
     <collision name="display">
-      <origin rpy="0 -0.3 0" xyz="0.97 0 0.785" />
-      <geometry>
-        <box size="0.06 0.225 0.375" />
+      <origin rpy="0 0 0" xyz="0.7275 0 0.64" />
+      <geometry>
+        <box size="0.126105200134 0.135 0.375982395822" />
       </geometry>
     </collision>
     <collision name="head_bearing_support">
-      <origin rpy="0 0 0" xyz="1.08 0 0.64" />
-      <geometry>
-        <box size="0.28 0.065 0.03" />
+      <origin rpy="0 0 0" xyz="0.81 0 0.495" />
+      <geometry>
+        <box size="0.21 0.039 0.03" />
       </geometry>
     </collision>
     <visual name="head_bearing_support">
-      <origin rpy="0 0 0" xyz="1.08 0 0.64" />
-      <geometry>
-        <box size="0.28 0.065 0.03" />
+      <origin rpy="0 0 0" xyz="0.81 0 0.495" />
+      <geometry>
+        <box size="0.21 0.039 0.03" />
       </geometry>
       <material name="bglx_aluminum">
@@ -55,19 +56,19 @@
     </visual>
     <collision name="sensor_mast">
-      <origin rpy="0 0 0" xyz="0.42 0 1.243" />
-      <geometry>
-        <box size="0.23 0.34 0.142" />
+      <origin rpy="0 0 0" xyz="0.315 0 1.098" />
+      <geometry>
+        <box size="0.1725 0.204 0.142" />
       </geometry>
     </collision>
     <collision name="terrain_camera_mount">
-      <origin rpy="0 0 0" xyz="1.005 0 0.855" />
-      <geometry>
-        <box size="0.095 0.07 0.025" />
+      <origin rpy="0 0 0" xyz="0.75375 0 0.71" />
+      <geometry>
+        <box size="0.07125 0.042 0.025" />
       </geometry>
     </collision>
     <visual name="terrain_camera_mount">
-      <origin rpy="0 0 0" xyz="1.005 0 0.855" />
-      <geometry>
-        <box size="0.095 0.07 0.025" />
+      <origin rpy="0 0 0" xyz="0.75375 0 0.71" />
+      <geometry>
+        <box size="0.07125 0.042 0.025" />
       </geometry>
       <material name="bglx_aluminum">
@@ -76,7 +77,7 @@
     </visual>
     <visual name="bglx_color_body_0">
-      <origin rpy="0 0 0" xyz="0 0 0" />
-      <geometry>
-        <mesh filename="package://etrike_description/meshes/concept_color/body_0.stl" scale="1 1 1" />
+      <origin rpy="0 0 0" xyz="0 0 -0.145" />
+      <geometry>
+        <mesh filename="package://etrike_description/meshes/concept_color/body_0.stl" scale="0.75 0.6 1" />
       </geometry>
       <material name="bglx_color_body_0">
@@ -85,7 +86,7 @@
     </visual>
     <visual name="bglx_color_body_1">
-      <origin rpy="0 0 0" xyz="0 0 0" />
-      <geometry>
-        <mesh filename="package://etrike_description/meshes/concept_color/body_1.stl" scale="1 1 1" />
+      <origin rpy="0 0 0" xyz="0 0 -0.145" />
+      <geometry>
+        <mesh filename="package://etrike_description/meshes/concept_color/body_1.stl" scale="0.75 0.6 1" />
       </geometry>
       <material name="bglx_color_body_1">
@@ -94,7 +95,7 @@
     </visual>
     <visual name="bglx_color_body_2">
-      <origin rpy="0 0 0" xyz="0 0 0" />
-      <geometry>
-        <mesh filename="package://etrike_description/meshes/concept_color/body_2.stl" scale="1 1 1" />
+      <origin rpy="0 0 0" xyz="0 0 -0.145" />
+      <geometry>
+        <mesh filename="package://etrike_description/meshes/concept_color/body_2.stl" scale="0.75 0.6 1" />
       </geometry>
       <material name="bglx_color_body_2">
@@ -103,7 +104,7 @@
     </visual>
     <visual name="bglx_color_body_3">
-      <origin rpy="0 0 0" xyz="0 0 0" />
-      <geometry>
-        <mesh filename="package://etrike_description/meshes/concept_color/body_3.stl" scale="1 1 1" />
+      <origin rpy="0 0 0" xyz="0 0 -0.145" />
+      <geometry>
+        <mesh filename="package://etrike_description/meshes/concept_color/body_3.stl" scale="0.75 0.6 1" />
       </geometry>
       <material name="bglx_color_body_3">
@@ -112,7 +113,7 @@
     </visual>
     <visual name="bglx_color_body_4">
-      <origin rpy="0 0 0" xyz="0 0 0" />
-      <geometry>
-        <mesh filename="package://etrike_description/meshes/concept_color/body_4.stl" scale="1 1 1" />
+      <origin rpy="0 0 0" xyz="0 0 -0.145" />
+      <geometry>
+        <mesh filename="package://etrike_description/meshes/concept_color/body_4.stl" scale="0.75 0.6 1" />
       </geometry>
       <material name="bglx_color_body_4">
@@ -121,7 +122,7 @@
     </visual>
     <visual name="bglx_color_body_5">
-      <origin rpy="0 0 0" xyz="0 0 0" />
-      <geometry>
-        <mesh filename="package://etrike_description/meshes/concept_color/body_5.stl" scale="1 1 1" />
+      <origin rpy="0 0 0" xyz="0 0 -0.145" />
+      <geometry>
+        <mesh filename="package://etrike_description/meshes/concept_color/body_5.stl" scale="0.75 0.6 1" />
       </geometry>
       <material name="bglx_color_body_5">
@@ -130,7 +131,7 @@
     </visual>
     <visual name="bglx_color_body_6">
-      <origin rpy="0 0 0" xyz="0 0 0" />
-      <geometry>
-        <mesh filename="package://etrike_description/meshes/concept_color/body_6.stl" scale="1 1 1" />
+      <origin rpy="0 0 0" xyz="0 0 -0.145" />
+      <geometry>
+        <mesh filename="package://etrike_description/meshes/concept_color/body_6.stl" scale="0.75 0.6 1" />
       </geometry>
       <material name="bglx_color_body_6">
@@ -139,7 +140,7 @@
     </visual>
     <visual name="bglx_color_body_7">
-      <origin rpy="0 0 0" xyz="0 0 0" />
-      <geometry>
-        <mesh filename="package://etrike_description/meshes/concept_color/body_7.stl" scale="1 1 1" />
+      <origin rpy="0 0 0" xyz="0 0 -0.145" />
+      <geometry>
+        <mesh filename="package://etrike_description/meshes/concept_color/body_7.stl" scale="0.75 0.6 1" />
       </geometry>
       <material name="bglx_color_body_7">
@@ -148,7 +149,7 @@
     </visual>
     <visual name="bglx_color_body_8">
-      <origin rpy="0 0 0" xyz="0 0 0" />
-      <geometry>
-        <mesh filename="package://etrike_description/meshes/concept_color/body_8.stl" scale="1 1 1" />
+      <origin rpy="0 0 0" xyz="0 0 -0.145" />
+      <geometry>
+        <mesh filename="package://etrike_description/meshes/concept_color/body_8.stl" scale="0.75 0.6 1" />
       </geometry>
       <material name="bglx_color_body_8">
@@ -157,7 +158,7 @@
     </visual>
     <visual name="bglx_color_body_9">
-      <origin rpy="0 0 0" xyz="0 0 0" />
-      <geometry>
-        <mesh filename="package://etrike_description/meshes/concept_color/body_9.stl" scale="1 1 1" />
+      <origin rpy="0 0 0" xyz="0 0 -0.145" />
+      <geometry>
+        <mesh filename="package://etrike_description/meshes/concept_color/body_9.stl" scale="0.75 0.6 1" />
       </geometry>
       <material name="bglx_color_body_9">
@@ -166,7 +167,7 @@
     </visual>
     <visual name="bglx_color_body_10">
-      <origin rpy="0 0 0" xyz="0 0 0" />
-      <geometry>
-        <mesh filename="package://etrike_description/meshes/concept_color/body_10.stl" scale="1 1 1" />
+      <origin rpy="0 0 0" xyz="0 0 -0.145" />
+      <geometry>
+        <mesh filename="package://etrike_description/meshes/concept_color/body_10.stl" scale="0.75 0.6 1" />
       </geometry>
       <material name="bglx_color_body_10">
@@ -174,4 +175,19 @@
       </material>
     </visual>
+    <visual name="prototype_rear_bumper">
+      <origin xyz="-0.185 0 0.16" rpy="0 0 0" />
+      <geometry>
+        <box size="0.03 0.42 0.04" />
+      </geometry>
+      <material name="prototype_bumper">
+        <color rgba="0.12 0.14 0.13 1" />
+      </material>
+    </visual>
+    <collision name="prototype_rear_bumper">
+      <origin xyz="-0.185 0 0.16" rpy="0 0 0" />
+      <geometry>
+        <box size="0.03 0.42 0.04" />
+      </geometry>
+    </collision>
   </link>
   <link name="base_footprint" />
@@ -183,36 +199,36 @@
   <link name="caster_mount">
     <inertial>
-      <origin rpy="0 0 0" xyz="-0.025 0 -0.19" />
-      <mass value="3" />
-      <inertia ixx="0.052" ixy="0" ixz="0" iyy="0.048" iyz="0" izz="0.015" />
+      <origin rpy="0 0 0" xyz="-0.01 0 -0.19" />
+      <mass value="2.93040293040293" />
+      <inertia ixx="0.04358776576958395" ixy="0.0" ixz="0.0" iyy="0.04237362637362638" iyz="0.0" izz="0.0029333091151272995" />
     </inertial>
     <collision name="fork_-1">
-      <origin rpy="0 -0.15 0" xyz="-0.025 -0.076 -0.215" />
-      <geometry>
-        <box size="0.047 0.047 0.3" />
+      <origin rpy="0 0 0" xyz="-0.01 -0.0359272727273 -0.215" />
+      <geometry>
+        <box size="0.036521472162 0.0222181818182 0.303654915607" />
       </geometry>
     </collision>
     <collision name="fork_1">
-      <origin rpy="0 -0.15 0" xyz="-0.025 0.076 -0.215" />
-      <geometry>
-        <box size="0.047 0.047 0.3" />
+      <origin rpy="0 0 0" xyz="-0.01 0.0359272727273 -0.215" />
+      <geometry>
+        <box size="0.036521472162 0.0222181818182 0.303654915607" />
       </geometry>
     </collision>
     <collision name="fork_crown">
-      <origin rpy="0 0 0" xyz="-0.07 0 -0.075" />
-      <geometry>
-        <box size="0.09 0.2 0.04" />
+      <origin rpy="0 0 0" xyz="-0.028 0 -0.075" />
+      <geometry>
+        <box size="0.036 0.0945454545455 0.04" />
       </geometry>
     </collision>
     <collision name="offset_fork_crown">
-      <origin rpy="0 0 0" xyz="-0.035 0 -0.075" />
-      <geometry>
-        <box size="0.15 0.07 0.038" />
+      <origin rpy="0 0 0" xyz="-0.014 0 -0.075" />
+      <geometry>
+        <box size="0.06 0.0330909090909 0.038" />
       </geometry>
     </collision>
     <visual name="offset_fork_crown">
-      <origin rpy="0 0 0" xyz="-0.035 0 -0.075" />
-      <geometry>
-        <box size="0.15 0.07 0.038" />
+      <origin rpy="0 0 0" xyz="-0.014 0 -0.075" />
+      <geometry>
+        <box size="0.06 0.0330909090909 0.038" />
       </geometry>
       <material name="bglx_aluminum">
@@ -221,67 +237,67 @@
     </visual>
     <collision name="mudguard_0">
-      <origin rpy="0 1.216818957 0" xyz="0.2814004365 0 -0.2610106046" />
-      <geometry>
-        <box size="0.101 0.12 0.016" />
+      <origin rpy="0 0 0" xyz="0.1125601746 0 -0.2610106046" />
+      <geometry>
+        <box size="0.0200071145597 0.0567272727273 0.100284248032" />
       </geometry>
     </collision>
     <collision name="mudguard_1">
-      <origin rpy="0 0.9088642179 0" xyz="0.2366418447 0 -0.1806073827" />
-      <geometry>
-        <box size="0.101 0.12 0.016" />
+      <origin rpy="0 0 0" xyz="0.09465673788 0 -0.1806073827" />
+      <geometry>
+        <box size="0.0298798984836 0.0567272727273 0.0895036939888" />
       </geometry>
     </collision>
     <collision name="mudguard_2">
-      <origin rpy="0 0.6009094786 0" xyz="0.1696178594 0 -0.117553477" />
-      <geometry>
-        <box size="0.101 0.12 0.016" />
+      <origin rpy="0 0 0" xyz="0.06784714376 0 -0.117553477" />
+      <geometry>
+        <box size="0.0369413127682 0.0567272727273 0.0703018272441" />
       </geometry>
     </collision>
     <collision name="mudguard_3">
-      <origin rpy="0 0.2929547393 0" xyz="0.08663470007 0 -0.07778156615" />
-      <geometry>
-        <box size="0.101 0.12 0.016" />
+      <origin rpy="0 0 0" xyz="0.034653880028 0 -0.07778156615" />
+      <geometry>
+        <box size="0.0405269560267 0.0567272727273 0.0444853321629" />
       </geometry>
     </collision>
     <collision name="mudguard_4">
-      <origin rpy="0 -0.015 0" xyz="-0.004499831252 0 -0.06503374937" />
-      <geometry>
-        <box size="0.101 0.12 0.016" />
+      <origin rpy="0 0 0" xyz="-0.0017999325008 0 -0.06503374937" />
+      <geometry>
+        <box size="0.0404914514853 0.0567272727273 0.0175131432219" />
       </geometry>
     </collision>
     <collision name="mudguard_5">
-      <origin rpy="0 -0.3229547393 0" xyz="-0.09521097797 0 -0.08050945591" />
-      <geometry>
-        <box size="0.101 0.12 0.016" />
+      <origin rpy="0 0 0" xyz="-0.038084391188 0 -0.08050945591" />
+      <geometry>
+        <box size="0.0403425608002 0.0567272727273 0.0472271916016" />
       </geometry>
     </collision>
     <collision name="mudguard_6">
-      <origin rpy="0 -0.6309094786 0" xyz="-0.1769638194 0 -0.1227525921" />
-      <geometry>
-        <box size="0.101 0.12 0.016" />
+      <origin rpy="0 0 0" xyz="-0.07078552776 0 -0.1227525921" />
+      <geometry>
+        <box size="0.0363978790767 0.0567272727273 0.0724976809436" />
       </geometry>
     </collision>
     <collision name="mudguard_7">
-      <origin rpy="0 -0.9388642179 0" xyz="-0.2420663127 0 -0.1877885437" />
-      <geometry>
-        <box size="0.101 0.12 0.016" />
+      <origin rpy="0 0 0" xyz="-0.09682652508 0 -0.1877885437" />
+      <geometry>
+        <box size="0.0290285574576 0.0567272727273 0.0909469362795" />
       </geometry>
     </collision>
     <collision name="mudguard_8">
-      <origin rpy="0 -1.246818957 0" xyz="-0.2843930297 0 -0.2694981432" />
-      <geometry>
-        <box size="0.101 0.12 0.016" />
+      <origin rpy="0 0 0" xyz="-0.11375721188 0 -0.2694981432" />
+      <geometry>
+        <box size="0.0189279680216 0.0567272727273 0.100839085696" />
       </geometry>
     </collision>
     <collision name="axle_sensor">
-      <origin rpy="0 0 0" xyz="0.035 0.145 -0.34" />
-      <geometry>
-        <box size="0.08 0.075 0.065" />
+      <origin rpy="0 0 0" xyz="0.014 0.0685454545455 -0.34" />
+      <geometry>
+        <box size="0.032 0.0354545454545 0.065" />
       </geometry>
     </collision>
     <visual name="bglx_color_steering_0">
-      <origin rpy="0 0 0" xyz="-0.07 0 0" />
-      <geometry>
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